Commit message: Add truck_description package, reduce spawn times, fix RViz truck orientation
- New truck_description package: dump truck URDF/xacro and meshes (GLB for Gazebo, STL for RViz)
- Spawn time reduction: excavator 6→4s, bridge 8→6s, controllers 9→7s, truck 8→6s
- RViz truck orientation: pete_visual_rpy arg (0 0 0 for STL) so truck matches Gazebo
- Gazebo spawn race fix: truck RSP remapped, truck group delayed for deterministic spawn
- README: updated log and quick start spawn times

Made-with: Cursor

File: src/excavator_description/urdf/truck.urdf.xacro (robot description, xacro)
@@ -1,7 +1,8 @@
 <?xml version="1.0"?>
 <robot name="truck" xmlns:xacro="http://ros.org/wiki/xacro">
+  <!-- Visual mesh extension: glb for Gazebo (textures), stl for RViz (Ogre loads STL reliably). -->
+  <xacro:arg name="pete_visual_ext" default="glb" />
   <xacro:property name="pi" value="3.1415926535897931" />
-  <!-- Pete articulated dump truck (GLB), Blender-exported truck only -->
-  <xacro:property name="pete_mesh_uri" value="package://excavator_description/meshes/truck/source/pete_dump_truck.glb" />
+  <xacro:property name="pete_mesh_uri" value="package://excavator_description/meshes/truck/source/pete_dump_truck.$(arg pete_visual_ext)" />
   <!-- Fallback: jsk_mbzirc_common (set use_pete to false in xacro or use mesh_uri for legacy) -->
   <xacro:property name="mesh_uri" value="package://jsk_mbzirc_common/gazebo_model/models/truck/meshes" />
