Commit message: AUWO digital twin: sensors, bridge, LiDAR frame fix, spawn fix
- Excavator: IMU + 3D LiDAR (gpu_lidar), visible sensor links (orange IMU, blue LiDAR)
- Worlds: default plugins (Physics, SceneBroadcaster, UserCommands), Imu + Sensors for sensor data
- Bridge: clock + /excavator/imu -> /imu, /excavator/points/points -> /points; GZ_PARTITION=auwo_sim
- points_frame_remap: /points -> /points_viz with frame_id sensor_lidar_link (fix RViz transform error)
- imu_to_pose: /imu -> /imu_pose for RViz orientation display
- Spawn: excavator from /robot_description, truck from file when spawn_dumper
- RViz: 3D LiDAR on /points_viz, IMU on /imu_pose; trajectory controller in controllers.yaml
- README: sensor viz, partition note; scripts/list_gz_sensor_topics.sh

Made-with: Cursor

File: src/excavator_description/urdf/excavator.urdf.xacro (robot description, xacro)
@@ -97,4 +97,48 @@
         <mesh filename="package://excavator_description/meshes/shovel.dae"/>
       </geometry>
+    </collision>
+  </link>
+  <!-- Sensor links (IMU and 3D LiDAR on body/cab) - visible physical sensor geometry -->
+  <link name="sensor_imu_link">
+    <inertial>
+      <mass value="0.02"/>
+      <origin xyz="0 0 0"/>
+      <inertia ixx="1e-5" iyy="1e-5" izz="1e-5" ixy="0" ixz="0" iyz="0"/>
+    </inertial>
+    <visual name="imu_visual">
+      <geometry><box size="0.12 0.10 0.03"/></geometry>
+      <origin xyz="0 0 0"/>
+      <material name="imu_material">
+        <color rgba="0.9 0.45 0.1 1"/>
+      </material>
+    </visual>
+    <collision name="imu_collision">
+      <geometry><box size="0.12 0.10 0.03"/></geometry>
+      <origin xyz="0 0 0"/>
+    </collision>
+  </link>
+  <link name="sensor_lidar_link">
+    <inertial>
+      <mass value="0.05"/>
+      <origin xyz="0 0 0"/>
+      <inertia ixx="1e-4" iyy="1e-4" izz="1e-4" ixy="0" ixz="0" iyz="0"/>
+    </inertial>
+    <visual name="lidar_base">
+      <geometry><cylinder radius="0.08" length="0.04"/></geometry>
+      <origin xyz="0 0 0" rpy="0 0 0"/>
+      <material name="lidar_base_material">
+        <color rgba="0.1 0.5 0.85 1"/>
+      </material>
+    </visual>
+    <visual name="lidar_dome">
+      <geometry><sphere radius="0.07"/></geometry>
+      <origin xyz="0 0 0.05" rpy="0 0 0"/>
+      <material name="lidar_dome_material">
+        <color rgba="0.2 0.6 0.9 0.95"/>
+      </material>
+    </visual>
+    <collision name="lidar_collision">
+      <geometry><cylinder radius="0.08" length="0.12"/></geometry>
+      <origin xyz="0 0 0.04" rpy="0 0 0"/>
     </collision>
   </link>
@@ -138,4 +182,15 @@
     <limit effort="3000.0" lower="-2.395" upper="-0.357" velocity="1.2"/>
   </joint>
+  <!-- Body -> sensor links (fixed, above cab) -->
+  <joint name="body_to_imu" type="fixed">
+    <parent link="body"/>
+    <child link="sensor_imu_link"/>
+    <origin xyz="0.3 0 0.25" rpy="0 0 0"/>
+  </joint>
+  <joint name="body_to_lidar" type="fixed">
+    <parent link="body"/>
+    <child link="sensor_lidar_link"/>
+    <origin xyz="0.35 0 0.4" rpy="0 0 0"/>
+  </joint>
   <!-- ros2_control interfaces -->
   <ros2_control name="GazeboSimSystem" type="system">
@@ -171,3 +226,56 @@
     </plugin>
   </gazebo>
+  <!-- IMU sensor (Gazebo Harmonic); orange so visible in sim -->
+  <gazebo reference="sensor_imu_link">
+    <material>Gazebo/Orange</material>
+    <sensor name="imu_sensor" type="imu">
+      <always_on>true</always_on>
+      <update_rate>100</update_rate>
+      <visualize>true</visualize>
+      <topic>/excavator/imu</topic>
+      <imu>
+        <angular_velocity>
+          <x><noise type="gaussian"><mean>0.0</mean><stddev>0.0002</stddev></noise></x>
+          <y><noise type="gaussian"><mean>0.0</mean><stddev>0.0002</stddev></noise></y>
+          <z><noise type="gaussian"><mean>0.0</mean><stddev>0.0002</stddev></noise></z>
+        </angular_velocity>
+        <linear_acceleration>
+          <x><noise type="gaussian"><mean>0.0</mean><stddev>0.017</stddev></noise></x>
+          <y><noise type="gaussian"><mean>0.0</mean><stddev>0.017</stddev></noise></y>
+          <z><noise type="gaussian"><mean>0.0</mean><stddev>0.017</stddev></noise></z>
+        </linear_acceleration>
+      </imu>
+    </sensor>
+  </gazebo>
+  <!-- 3D LiDAR sensor (gpu_lidar, Gazebo Harmonic); blue so visible in sim -->
+  <gazebo reference="sensor_lidar_link">
+    <material>Gazebo/Blue</material>
+    <sensor name="lidar_sensor" type="gpu_lidar">
+      <always_on>true</always_on>
+      <update_rate>10</update_rate>
+      <visualize>true</visualize>
+      <topic>/excavator/points</topic>
+      <lidar>
+        <scan>
+          <horizontal>
+            <samples>360</samples>
+            <resolution>1.0</resolution>
+            <min_angle>-3.14159265</min_angle>
+            <max_angle>3.14159265</max_angle>
+          </horizontal>
+          <vertical>
+            <samples>32</samples>
+            <resolution>1.0</resolution>
+            <min_angle>-0.261799</min_angle>
+            <max_angle>0.261799</max_angle>
+          </vertical>
+        </scan>
+        <range>
+          <min>0.2</min>
+          <max>30.0</max>
+          <resolution>0.01</resolution>
+        </range>
+      </lidar>
+    </sensor>
+  </gazebo>
 </robot>

Commit message: Stabilize headless MoveIt execution and Gazebo clock bridging.
Use explicit trajectory_execution tolerance config, separate and harden clock/sensor bridges for headless Gazebo, and relax shovel joint bounds so plan/execute no longer fails from start-state drift.

Made-with: Cursor

File: src/excavator_description/urdf/excavator.urdf.xacro (robot description, xacro)
@@ -180,5 +180,6 @@
     <origin xyz="-1.362 0 -0.154"/>
     <dynamics damping="6.0" friction="0.8"/>
-    <limit effort="3000.0" lower="-2.395" upper="-0.357" velocity="1.2"/>
+    <!-- Lower bound slightly below nominal URDF so Gazebo start pose / solver drift stays inside MoveIt bounds -->
+    <limit effort="3000.0" lower="-2.60" upper="-0.357" velocity="1.2"/>
   </joint>
   <!-- Body -> sensor links (fixed, above cab) -->

Commit message: feat: add MoveIt config package and Gazebo planning integration

File: src/excavator_description/urdf/excavator.urdf.xacro (robot description, xacro)
@@ -1,4 +1,6 @@
 <?xml version="1.0"?>
 <robot name="excavator" xmlns:xacro="http://www.ros.org/wiki/xacro">
+  <!-- When true: mock_components/GenericSystem for RViz-only MoveIt (no Gazebo). -->
+  <xacro:arg name="use_mock_hardware" default="false"/>
   <xacro:property name="mesh_uri" value="package://excavator_description/meshes"/>
   <!-- Massless root -->
@@ -150,5 +152,8 @@
   </joint>
   <!-- Joints with damping/friction and stronger limits -->
-  <joint name="body_rotation" type="continuous">
+  <!-- Revolute with wide limits (not continuous): MoveIt + JointTrajectoryController validate the
+       first waypoint against /joint_states; continuous joints often report large accumulated
+       angles while planned trajectories use a different branch → instant "start deviates" abort. -->
+  <joint name="body_rotation" type="revolute">
     <parent link="base"/>
     <child link="body"/>
@@ -156,5 +161,5 @@
     <origin xyz="0.0 0.0 0.6"/>
     <dynamics damping="8.0" friction="0.5"/>
-    <limit effort="4000.0" velocity="1.5"/>
+    <limit effort="4000.0" lower="-12.566370614359172" upper="12.566370614359172" velocity="1.5"/>
   </joint>
   <joint name="arm1_rotation" type="revolute">
@@ -180,6 +185,6 @@
     <origin xyz="-1.362 0 -0.154"/>
     <dynamics damping="6.0" friction="0.8"/>
-    <!-- Lower bound slightly below nominal URDF so Gazebo start pose / solver drift stays inside MoveIt bounds -->
-    <limit effort="3000.0" lower="-2.60" upper="-0.357" velocity="1.2"/>
+    <!-- Upper relaxed toward 0: gz/joint_states often ~-0.01 rad; tight upper=-0.357 made CheckStartStateBounds fail. -->
+    <limit effort="3000.0" lower="-2.60" upper="0.35" velocity="1.2"/>
   </joint>
   <!-- Body -> sensor links (fixed, above cab) -->
@@ -194,37 +199,90 @@
     <origin xyz="0.35 0 0.4" rpy="0 0 0"/>
   </joint>
-  <!-- ros2_control interfaces -->
-  <ros2_control name="GazeboSimSystem" type="system">
-    <hardware>
-      <plugin>gz_ros2_control/GazeboSimSystem</plugin>
-    </hardware>
+  <!-- Mock hardware defaults all states to 0; arm joints must be negative per URDF limits. -->
+  <xacro:macro name="excavator_mock_ros2_control_joints">
     <joint name="body_rotation">
       <command_interface name="position"/>
-      <state_interface name="position"/>
+      <state_interface name="position">
+        <param name="initial_value">0.0</param>
+      </state_interface>
       <state_interface name="velocity"/>
     </joint>
     <joint name="arm1_rotation">
       <command_interface name="position"/>
-      <state_interface name="position"/>
+      <state_interface name="position">
+        <param name="initial_value">-0.70</param>
+      </state_interface>
       <state_interface name="velocity"/>
     </joint>
     <joint name="arm2_rotation">
       <command_interface name="position"/>
-      <state_interface name="position"/>
+      <state_interface name="position">
+        <param name="initial_value">-1.26</param>
+      </state_interface>
       <state_interface name="velocity"/>
     </joint>
     <joint name="shovel_rotation">
       <command_interface name="position"/>
-      <state_interface name="position"/>
-      <state_interface name="velocity"/>
-    </joint>
-  </ros2_control>
-  <!-- Gazebo ros2_control plugin -->
-  <gazebo>
-    <plugin filename="libgz_ros2_control-system.so"
-            name="gz_ros2_control::GazeboSimROS2ControlPlugin">
-      <parameters>$(find excavator_description)/config/controllers.yaml</parameters>
-    </plugin>
-  </gazebo>
+      <state_interface name="position">
+        <param name="initial_value">-1.12</param>
+      </state_interface>
+      <state_interface name="velocity"/>
+    </joint>
+  </xacro:macro>
+  <xacro:macro name="excavator_ros2_control_joints">
+    <joint name="body_rotation">
+      <command_interface name="position"/>
+      <state_interface name="position">
+        <param name="initial_value">0.0</param>
+      </state_interface>
+      <state_interface name="velocity"/>
+    </joint>
+    <joint name="arm1_rotation">
+      <command_interface name="position"/>
+      <state_interface name="position">
+        <param name="initial_value">-0.70</param>
+      </state_interface>
+      <state_interface name="velocity"/>
+    </joint>
+    <joint name="arm2_rotation">
+      <command_interface name="position"/>
+      <state_interface name="position">
+        <param name="initial_value">-1.26</param>
+      </state_interface>
+      <state_interface name="velocity"/>
+    </joint>
+    <joint name="shovel_rotation">
+      <command_interface name="position"/>
+      <state_interface name="position">
+        <param name="initial_value">-1.12</param>
+      </state_interface>
+      <state_interface name="velocity"/>
+    </joint>
+  </xacro:macro>
+  <!-- ros2_control: Gazebo sim hardware (default) or mock hardware (RViz-only demo). -->
+  <xacro:unless value="$(arg use_mock_hardware)">
+    <ros2_control name="GazeboSimSystem" type="system">
+      <hardware>
+        <plugin>gz_ros2_control/GazeboSimSystem</plugin>
+      </hardware>
+      <xacro:excavator_ros2_control_joints/>
+    </ros2_control>
+    <gazebo>
+      <plugin filename="libgz_ros2_control-system.so"
+              name="gz_ros2_control::GazeboSimROS2ControlPlugin">
+        <parameters>$(find excavator_description)/config/controllers.yaml</parameters>
+      </plugin>
+    </gazebo>
+  </xacro:unless>
+  <xacro:if value="$(arg use_mock_hardware)">
+    <ros2_control name="MockHardwareSystem" type="system">
+      <hardware>
+        <plugin>mock_components/GenericSystem</plugin>
+        <param name="mock_sensor_commands">false</param>
+        <param name="position_state_following_offset">0.0</param>
+      </hardware>
+      <xacro:excavator_mock_ros2_control_joints/>
+    </ros2_control>
+  </xacro:if>
   <!-- IMU sensor (Gazebo Harmonic); orange so visible in sim -->
   <gazebo reference="sensor_imu_link">

Commit message: feat: boom/stick/bucket excavator rename, MoveIt world TF, Gazebo pause, environment.stl

File: src/excavator_description/urdf/excavator.urdf.xacro (robot description, xacro)
@@ -45,5 +45,5 @@
   </link>
   <!-- ARM1 (boom) -->
-  <link name="arm1">
+  <link name="boom">
     <inertial>
       <mass value="120.0"/>
@@ -53,16 +53,16 @@
     <visual>
       <geometry>
-        <mesh filename="package://excavator_description/meshes/arm1.dae"/>
-      </geometry>
-      <origin xyz="0 0 0"/>
-    </visual>
-    <collision>
-      <geometry>
-        <mesh filename="package://excavator_description/meshes/arm1.dae"/>
+        <mesh filename="package://excavator_description/meshes/boom.dae"/>
+      </geometry>
+      <origin xyz="0 0 0"/>
+    </visual>
+    <collision>
+      <geometry>
+        <mesh filename="package://excavator_description/meshes/boom.dae"/>
       </geometry>
     </collision>
   </link>
   <!-- ARM2 (stick) -->
-  <link name="arm2">
+  <link name="stick">
     <inertial>
       <mass value="80.0"/>
@@ -72,16 +72,16 @@
     <visual>
       <geometry>
-        <mesh filename="package://excavator_description/meshes/arm2.dae"/>
-      </geometry>
-      <origin xyz="0 0 0"/>
-    </visual>
-    <collision>
-      <geometry>
-        <mesh filename="package://excavator_description/meshes/arm2.dae"/>
+        <mesh filename="package://excavator_description/meshes/stick.dae"/>
+      </geometry>
+      <origin xyz="0 0 0"/>
+    </visual>
+    <collision>
+      <geometry>
+        <mesh filename="package://excavator_description/meshes/stick.dae"/>
       </geometry>
     </collision>
   </link>
   <!-- SHOVEL (bucket) -->
-  <link name="shovel">
+  <link name="bucket">
     <inertial>
       <mass value="60.0"/>
@@ -91,11 +91,11 @@
     <visual>
       <geometry>
-        <mesh filename="package://excavator_description/meshes/shovel.dae"/>
-      </geometry>
-      <origin xyz="0 0 0"/>
-    </visual>
-    <collision>
-      <geometry>
-        <mesh filename="package://excavator_description/meshes/shovel.dae"/>
+        <mesh filename="package://excavator_description/meshes/bucket.dae"/>
+      </geometry>
+      <origin xyz="0 0 0"/>
+    </visual>
+    <collision>
+      <geometry>
+        <mesh filename="package://excavator_description/meshes/bucket.dae"/>
       </geometry>
     </collision>
@@ -163,7 +163,7 @@
     <limit effort="4000.0" lower="-12.566370614359172" upper="12.566370614359172" velocity="1.5"/>
   </joint>
-  <joint name="arm1_rotation" type="revolute">
+  <joint name="boom_rotation" type="revolute">
     <parent link="body"/>
-    <child link="arm1"/>
+    <child link="boom"/>
     <axis xyz="0 1 0"/>
     <origin xyz="0.933 -0.134 0.302"/>
@@ -171,7 +171,7 @@
     <limit effort="4000.0" lower="-1.308" upper="-0.087" velocity="1.0"/>
   </joint>
-  <joint name="arm2_rotation" type="revolute">
-    <parent link="arm1"/>
-    <child link="arm2"/>
+  <joint name="stick_rotation" type="revolute">
+    <parent link="boom"/>
+    <child link="stick"/>
     <axis xyz="0 1 0"/>
     <origin xyz="2.586 0 -0.625"/>
@@ -179,7 +179,7 @@
     <limit effort="3500.0" lower="-2.428" upper="-0.085" velocity="1.0"/>
   </joint>
-  <joint name="shovel_rotation" type="revolute">
-    <parent link="arm2"/>
-    <child link="shovel"/>
+  <joint name="bucket_rotation" type="revolute">
+    <parent link="stick"/>
+    <child link="bucket"/>
     <axis xyz="0 1 0"/>
     <origin xyz="-1.362 0 -0.154"/>
@@ -208,5 +208,5 @@
       <state_interface name="velocity"/>
     </joint>
-    <joint name="arm1_rotation">
+    <joint name="boom_rotation">
       <command_interface name="position"/>
       <state_interface name="position">
@@ -215,5 +215,5 @@
       <state_interface name="velocity"/>
     </joint>
-    <joint name="arm2_rotation">
+    <joint name="stick_rotation">
       <command_interface name="position"/>
       <state_interface name="position">
@@ -222,5 +222,5 @@
       <state_interface name="velocity"/>
     </joint>
-    <joint name="shovel_rotation">
+    <joint name="bucket_rotation">
       <command_interface name="position"/>
       <state_interface name="position">
@@ -238,5 +238,5 @@
       <state_interface name="velocity"/>
     </joint>
-    <joint name="arm1_rotation">
+    <joint name="boom_rotation">
       <command_interface name="position"/>
       <state_interface name="position">
@@ -245,5 +245,5 @@
       <state_interface name="velocity"/>
     </joint>
-    <joint name="arm2_rotation">
+    <joint name="stick_rotation">
       <command_interface name="position"/>
       <state_interface name="position">
@@ -252,5 +252,5 @@
       <state_interface name="velocity"/>
     </joint>
-    <joint name="shovel_rotation">
+    <joint name="bucket_rotation">
       <command_interface name="position"/>
       <state_interface name="position">

Commit message: Add physical twin config, tf dump, and update URDF/launch files

File: src/excavator_description/urdf/excavator.urdf.xacro (robot description, xacro)
@@ -17,5 +17,5 @@
         <mesh filename="package://excavator_description/meshes/base.dae"/>
       </geometry>
-      <origin xyz="0 0 0"/>
+      <origin xyz="0 0 0" />
     </visual>
     <collision>
@@ -36,5 +36,5 @@
         <mesh filename="package://excavator_description/meshes/body.dae"/>
       </geometry>
-      <origin xyz="0 0 0"/>
+      <origin xyz="0 0 0" />
     </visual>
     <collision>
@@ -55,5 +55,5 @@
         <mesh filename="package://excavator_description/meshes/boom.dae"/>
       </geometry>
-      <origin xyz="0 0 0"/>
+      <origin xyz="0 0 0" />
     </visual>
     <collision>
@@ -74,5 +74,5 @@
         <mesh filename="package://excavator_description/meshes/stick.dae"/>
       </geometry>
-      <origin xyz="0 0 0"/>
+      <origin xyz="0 0 0" />
     </visual>
     <collision>
@@ -93,5 +93,5 @@
         <mesh filename="package://excavator_description/meshes/bucket.dae"/>
       </geometry>
-      <origin xyz="0 0 0"/>
+      <origin xyz="0 0 0" rpy="0 3.14159 0"/>
     </visual>
     <collision>
@@ -128,5 +128,5 @@
     <visual name="lidar_base">
       <geometry><cylinder radius="0.08" length="0.04"/></geometry>
-      <origin xyz="0 0 0" rpy="0 0 0"/>
+      <origin xyz="0 0 0" rpy="0 0 3.14159"/>
       <material name="lidar_base_material">
         <color rgba="0.1 0.5 0.85 1"/>
@@ -149,5 +149,5 @@
     <parent link="base_link"/>
     <child link="base"/>
-    <origin xyz="0 0 0" rpy="0 0 0"/>
+    <origin xyz="0 0 0" rpy="0 0 3.14159"/>
   </joint>
   <!-- Joints with damping/friction and stronger limits -->
@@ -169,5 +169,5 @@
     <origin xyz="0.933 -0.134 0.302"/>
     <dynamics damping="10.0" friction="1.5"/>
-    <limit effort="4000.0" lower="-1.308" upper="-0.087" velocity="1.0"/>
+    <limit effort="4000.0" lower="-1.40" upper="0.20" velocity="1.0"/>
   </joint>
   <joint name="stick_rotation" type="revolute">
@@ -177,5 +177,5 @@
     <origin xyz="2.586 0 -0.625"/>
     <dynamics damping="8.0" friction="1.2"/>
-    <limit effort="3500.0" lower="-2.428" upper="-0.085" velocity="1.0"/>
+    <limit effort="3500.0" lower="-2.428" upper="0.20" velocity="1.0"/>
   </joint>
   <joint name="bucket_rotation" type="revolute">
@@ -186,5 +186,5 @@
     <dynamics damping="6.0" friction="0.8"/>
     <!-- Upper relaxed toward 0: gz/joint_states often ~-0.01 rad; tight upper=-0.357 made CheckStartStateBounds fail. -->
-    <limit effort="3000.0" lower="-2.60" upper="0.35" velocity="1.2"/>
+    <limit effort="3000.0" lower="-2.00" upper="2.00" velocity="1.2"/>
   </joint>
   <!-- Body -> sensor links (fixed, above cab) -->
